Commit message: Update Roula's description

File: src/jaguar_description/urdf/model.urdf (robot description, URDF)
Before this commit: robot jaguar_robot, 8 links, 7 joints
Links:
- removed link base_footprint
Joints:
- removed joint base_footprint_joint
- joint imu_joint: origin xyz=0 0 0.149 rpy=0 -1.5708 3.1416 -> xyz=0 0 0.175 rpy=0 0 0
